Commit message: Fix wheel axis rotation in RVIZ.

File: src/wave_rover_description/urdf/rover.urdf.xacro (robot description, xacro)
@@ -136,10 +136,10 @@
    <origin xyz="0 0 0" rpy="-1.5708 0 -1.5708"/>
  </joint>
- <!-- Wheel Links (unchanged) -->
+ <!-- Wheel Links -->
  <!-- Front Left Wheel -->
  <link name="front_left_wheel">
    <xacro:inertia_wheel/>
    <collision>
-     <origin rpy="1.5708 0 0" xyz="0 0 0"/>
+     <origin rpy="1.5708 0 0" xyz="0.061 0.050 ${z_offset}"/>
      <geometry>
        <cylinder length="${wheel_length}" radius="${wheel_radius}"/>
@@ -155,86 +155,86 @@
  </link>
  <joint name="front_left_wheel_joint" type="revolute">
+   <parent link="base_link"/>
+   <child link="back_right_wheel"/>
+   <origin xyz="-0.061 -0.050 ${z_offset}" rpy="0 0 0"/>
+   <axis xyz="1 0 0">
+     <dynamics damping="1.0" friction="1.0"/>
+   </axis>
+   <limit lower="-1000" upper="1000" effort="10.0" velocity="10.0"/>
+ </joint>
+ <!-- Front Right Wheel -->
+ <link name="front_right_wheel">
+   <xacro:inertia_wheel/>
+   <collision>
+     <origin rpy="1.5708 0 0" xyz="0.061 -0.050 ${z_offset}"/>
+     <geometry>
+       <cylinder length="${wheel_length}" radius="${wheel_radius}"/>
+     </geometry>
+   </collision>
+   <visual>
+     <origin rpy="1.570795 0 0" xyz="0 0 0"/>
+     <geometry>
+       <mesh filename="package://wave_rover_description/meshes/rightside_wheel.stl" scale="0.001 0.001 0.001"/>
+     </geometry>
+     <material name="black"/>
+   </visual>
+ </link>
+ <joint name="front_right_wheel_joint" type="revolute">
+   <parent link="base_link"/>
+   <child link="front_right_wheel"/>
+   <origin xyz="0.061 -0.050 ${z_offset}" rpy="0 0 0"/>
+   <axis xyz="1 0 0">
+     <dynamics damping="1.0" friction="1.0"/>
+   </axis>
+   <limit lower="-1000" upper="1000" effort="10.0" velocity="10.0"/>
+ </joint>
+ <!-- Back Left Wheel -->
+ <link name="back_left_wheel">
+   <xacro:inertia_wheel/>
+   <collision>
+     <origin rpy="1.5708 0 0" xyz="-0.061 0.050 ${z_offset}"/>
+     <geometry>
+       <cylinder length="${wheel_length}" radius="${wheel_radius}"/>
+     </geometry>
+   </collision>
+   <visual>
+     <origin rpy="1.570795 0 0" xyz="0 0 0"/>
+     <geometry>
+       <mesh filename="package://wave_rover_description/meshes/leftside_wheel.stl" scale="0.001 0.001 0.001"/>
+     </geometry>
+     <material name="black"/>
+   </visual>
+ </link>
+ <joint name="back_left_wheel_joint" type="revolute">
+   <parent link="base_link"/>
+   <child link="back_left_wheel"/>
+   <origin xyz="-0.061 0.050 ${z_offset}" rpy="0 0 0"/>
+   <axis xyz="1 0 0">
+     <dynamics damping="1.0" friction="1.0"/>
+   </axis>
+   <limit lower="-1000" upper="1000" effort="10.0" velocity="10.0"/>
+ </joint>
+ <!-- Back Right Wheel -->
+ <link name="back_right_wheel">
+   <xacro:inertia_wheel/>
+   <collision>
+     <origin rpy="1.5708 0 0" xyz="-0.061 -0.050 ${z_offset}"/>
+     <geometry>
+       <cylinder length="${wheel_length}" radius="${wheel_radius}"/>
+     </geometry>
+   </collision>
+   <visual>
+     <origin rpy="1.570795 0 0" xyz="0 0 0"/>
+     <geometry>
+       <mesh filename="package://wave_rover_description/meshes/rightside_wheel.stl" scale="0.001 0.001 0.001"/>
+     </geometry>
+     <material name="black"/>
+   </visual>
+ </link>
+  <joint name="back_right_wheel_joint" type="revolute">
    <parent link="base_link"/>
    <child link="front_left_wheel"/>
    <origin xyz="0.061 0.050 ${z_offset}" rpy="0 0 0"/>
-   <axis xyz="0 1 0">
-     <dynamics damping="1.0" friction="1.0"/>
-   </axis>
-   <limit lower="-1000" upper="1000" effort="10.0" velocity="10.0"/>
- </joint>
- <!-- Front Right Wheel -->
- <link name="front_right_wheel">
-   <xacro:inertia_wheel/>
-   <collision>
-     <origin rpy="1.5708 0 0" xyz="0 0 0"/>
-     <geometry>
-       <cylinder length="${wheel_length}" radius="${wheel_radius}"/>
-     </geometry>
-   </collision>
-   <visual>
-     <origin rpy="1.570795 0 0" xyz="0 0 0"/>
-     <geometry>
-       <mesh filename="package://wave_rover_description/meshes/rightside_wheel.stl" scale="0.001 0.001 0.001"/>
-     </geometry>
-     <material name="black"/>
-   </visual>
- </link>
- <joint name="front_right_wheel_joint" type="revolute">
-   <parent link="base_link"/>
-   <child link="front_right_wheel"/>
-   <origin xyz="0.061 -0.050 ${z_offset}" rpy="0 0 0"/>
-   <axis xyz="0 1 0">
-     <dynamics damping="1.0" friction="1.0"/>
-   </axis>
-   <limit lower="-1000" upper="1000" effort="10.0" velocity="10.0"/>
- </joint>
- <!-- Back Left Wheel -->
- <link name="back_left_wheel">
-   <xacro:inertia_wheel/>
-   <collision>
-     <origin rpy="1.5708 0 0" xyz="0 0 0"/>
-     <geometry>
-       <cylinder length="${wheel_length}" radius="${wheel_radius}"/>
-     </geometry>
-   </collision>
-   <visual>
-     <origin rpy="1.570795 0 0" xyz="0 0 0"/>
-     <geometry>
-       <mesh filename="package://wave_rover_description/meshes/leftside_wheel.stl" scale="0.001 0.001 0.001"/>
-     </geometry>
-     <material name="black"/>
-   </visual>
- </link>
- <joint name="back_left_wheel_joint" type="revolute">
-   <parent link="base_link"/>
-   <child link="back_left_wheel"/>
-   <origin xyz="-0.061 0.050 ${z_offset}" rpy="0 0 0"/>
-   <axis xyz="0 1 0">
-     <dynamics damping="1.0" friction="1.0"/>
-   </axis>
-   <limit lower="-1000" upper="1000" effort="10.0" velocity="10.0"/>
- </joint>
- <!-- Back Right Wheel -->
- <link name="back_right_wheel">
-   <xacro:inertia_wheel/>
-   <collision>
-     <origin rpy="1.5708 0 0" xyz="0 0 0"/>
-     <geometry>
-       <cylinder length="${wheel_length}" radius="${wheel_radius}"/>
-     </geometry>
-   </collision>
-   <visual>
-     <origin rpy="1.570795 0 0" xyz="0 0 0"/>
-     <geometry>
-       <mesh filename="package://wave_rover_description/meshes/rightside_wheel.stl" scale="0.001 0.001 0.001"/>
-     </geometry>
-     <material name="black"/>
-   </visual>
- </link>
- <joint name="back_right_wheel_joint" type="revolute">
-   <parent link="base_link"/>
-   <child link="back_right_wheel"/>
-   <origin xyz="-0.061 -0.050 ${z_offset}" rpy="0 0 0"/>
-   <axis xyz="0 1 0">
+   <axis xyz="1 0 0">
      <dynamics damping="1.0" friction="1.0"/>
    </axis>

Commit message: Fix wheels in urdf.

File: src/wave_rover_description/urdf/rover.urdf.xacro (robot description, xacro)
@@ -156,5 +156,5 @@
  <joint name="front_left_wheel_joint" type="revolute">
    <parent link="base_link"/>
-   <child link="back_right_wheel"/>
+   <child link="front_left_wheel"/>
    <origin xyz="-0.061 -0.050 ${z_offset}" rpy="0 0 0"/>
    <axis xyz="1 0 0">
@@ -234,5 +234,5 @@
   <joint name="back_right_wheel_joint" type="revolute">
    <parent link="base_link"/>
-   <child link="front_left_wheel"/>
+   <child link="back_right_wheel"/>
    <origin xyz="0.061 0.050 ${z_offset}" rpy="0 0 0"/>
    <axis xyz="1 0 0">
